File: Janus HW/Janus HW.kicad_sch (KiCad schematic)
At the start: 20 parts, among them IC1 ESP32-C6FH4, IC2 UM980, IC3 MP2338GTL-P, J1 USB_B_Micro, U2 RFM69HCW

Commit message: Fiddling in Kicad
Parts:
- removed IC1: ESP32-C6FH4, footprints:QFN50P500X500X90-33N, symbol SamacSys_Parts:ESP32-C6FH4
- added C9: 100nF, Capacitor_SMD:C_0201_0603Metric_Pad0.64x0.40mm_HandSolder, symbol Device:C
- added J2: Conn_Coaxial_Small, Connector_Coaxial:U.FL_Molex_MCRF_73412-0110_Vertical, symbol Connector:Conn_Coaxial_Small
- added U1: ESP32-C3-MINI-1U-N4, footprints:XCVR_ESP32-C3-MINI-1U-N4, symbol ESP32-C3-MINI-1U-N4:ESP32-C3-MINI-1U-N4
- IC3: footprint SOTFL50P160X60-8N -> SamacSys_Parts:SOTFL50P160X60-8N
Connections:
- net +3.3V: now also C9.2, U1.3 (3V3)
- net GND: now also C9.1, J2.2 (Ext), U1.1 (GND), U1.11 (GND__2), U1.14 (GND__3), U1.2 (GND__1), U1.36 (GND__4), U1.37 (GND__5), U1.38 (GND__6), U1.39 (GND__7), U1.40 (GND__8), U1.41 (GND__9), U1.42 (GND__10), U1.43 (GND__11), U1.44 (GND__12), U1.45 (GND__13), U1.46 (GND__14), U1.47 (GND__15), U1.48 (GND__16), U1.49_1 (GND__17), U1.49_2 (GND__18), U1.49_3 (GND__19), U1.49_4 (GND__20), U1.49_5 (GND__21), U1.49_6 (GND__22), U1.49_7 (GND__23), U1.49_8 (GND__24), U1.49_9 (GND__25), U1.50 (GND__26), U1.51 (GND__27), U1.52 (GND__28), U1.53 (GND__29)
- net GPSRX: now also U1.31 (TXD0)
- net GPSTX: now also U1.30 (RXD0)
- net SPI_MISO: now also U1.16 (IO10)
- net SPI_MOSI: now also U1.13 (IO1)
- net SPI_SCK: now also U1.12 (IO0)
- net USB+: now also U1.27 (IO19)
- net USB-: now also U1.26 (IO18)
- net ANTFRM: no longer names the net of U2.9 (ANT)
- net ANTFRM: now also J2.1 (In)
- net ANTGPS: no longer names the net of AE2.1 (A), C1.2, L1.2
- net ANTUM980: no longer names the net of C1.1, IC2.2 (ANT_IN)
- net SPI_DIO0 renamed SPI_INT
- net SPI_INT: now also U1.6 (IO3)
- net SPI_NSS renamed SPI_CS
- net SPI_CS: now also U1.18 (IO4)
- no-connect marks 24 -> 56
Other:
- moved on the sheet: AE2, C1, C2, C3, C4, C5, C8, IC2, L1
